Commit message: fix some bug

File: turtlebot/turtlebot_description/urdf/stacks/hexagons.urdf.xacro (robot description, xacro)
@@ -3,5 +3,6 @@
   Hexagon stacks
  -->
-<robot name="stack_hexagons" xmlns:xacro="http://ros.org/wiki/xacro">
+<robot name="stack_hexagons"
+  xmlns:xacro="http://ros.org/wiki/xacro">
   <xacro:include filename="$(find turtlebot_description)/urdf/common_properties.urdf.xacro"/>
   <!-- Xacro properties -->
@@ -31,7 +32,5 @@
         <mass value="0.008"/>
         <origin xyz="0 0 0" rpy="0 0 0"/>
-        <inertia ixx="0.000001686" ixy="0.0" ixz="0.0"
-                 iyy="0.000001686" iyz="0.0"
-                 izz="0.000000144"/>
+        <inertia ixx="0.000001686" ixy="0.0" ixz="0.0" iyy="0.000001686" iyz="0.0" izz="0.000000144"/>
       </inertial>
     </link>
@@ -59,7 +58,5 @@
         <mass value="0.012"/>
         <origin xyz="0 0 0"/>
-        <inertia ixx="0.000003805" ixy="0.0" ixz="0.0"
-                 iyy="0.000003805" iyz="0.0"
-                 izz="0.000000216"/>
+        <inertia ixx="0.000003805" ixy="0.0" ixz="0.0" iyy="0.000003805" iyz="0.0" izz="0.000000216"/>
       </inertial>
     </link>
@@ -87,7 +84,5 @@
         <mass value="0.060"/>
         <origin xyz="0 0 0"/>
-        <inertia ixx="0.000206991" ixy="0.0" ixz="0.0"
-                 iyy="0.000206991" iyz="0.0"
-                 izz="0.000001080"/>
+        <inertia ixx="0.000206991" ixy="0.0" ixz="0.0" iyy="0.000206991" iyz="0.0" izz="0.000001080"/>
       </inertial>
     </link>
@@ -115,7 +110,5 @@
         <mass value="0.020"/>
         <origin xyz="0 0 0"/>
-        <inertia ixx="0.000014782" ixy="0.0" ixz="0.0"
-                 iyy="0.000014782" iyz="0.0"
-                 izz="0.000000360"/>
+        <inertia ixx="0.000014782" ixy="0.0" ixz="0.0" iyy="0.000014782" iyz="0.0" izz="0.000000360"/>
       </inertial>
     </link>
@@ -154,7 +147,5 @@
         <mass value="0.520" />
         <origin xyz="0 0 0" />
-        <inertia ixx="0.003328" ixy="0.0" ixz="0.0"
-                 iyy="0.003328" iyz="0.0"
-                 izz="0.006656" />
+        <inertia ixx="0.003328" ixy="0.0" ixz="0.0" iyy="0.003328" iyz="0.0" izz="0.006656" />
       </inertial>
     </link>
@@ -178,6 +169,5 @@
         <origin xyz="0.01364 0.0 0.0" rpy="0 0 0"/>
         <geometry>
-          <mesh filename="package://turtlebot_description/meshes/stacks/hexagons/plate_simple.stl"
-                scale="${M_SCALE} ${M_SCALE} ${M_SCALE}"/>
+          <mesh filename="package://turtlebot_description/meshes/stacks/hexagons/plate_simple.stl" scale="${M_SCALE} ${M_SCALE} ${M_SCALE}"/>
         </geometry>
       </collision>
@@ -185,7 +175,5 @@
         <mass value="0.520" />
         <origin xyz="0 0 0" />
-        <inertia ixx="0.003328" ixy="0.0" ixz="0.0"
-                 iyy="0.003328" iyz="0.0"
-                 izz="0.006656" />
+        <inertia ixx="0.003328" ixy="0.0" ixz="0.0" iyy="0.003328" iyz="0.0" izz="0.006656" />
       </inertial>
     </link>
@@ -211,6 +199,5 @@
         <origin xyz="0.01364 0 0" rpy="0 0 0"/>
         <geometry>
-          <mesh filename="package://turtlebot_description/meshes/stacks/hexagons/plate_simple.stl"
-                scale="${M_SCALE} ${M_SCALE} ${M_SCALE}"/>
+          <mesh filename="package://turtlebot_description/meshes/stacks/hexagons/plate_simple.stl" scale="${M_SCALE} ${M_SCALE} ${M_SCALE}"/>
         </geometry>
       </collision>
@@ -218,9 +205,19 @@
         <mass value="0.520"/>
         <origin xyz="0 0 0"/>
-        <inertia ixx="0.003328" ixy="0.0" ixz="0.0"
-                 iyy="0.003328" iyz="0.0"
-                 izz="0.006656" />
-      </inertial>
-    </link>
-  </xacro:macro>
+        <inertia ixx="0.003328" ixy="0.0" ixz="0.0" iyy="0.003328" iyz="0.0" izz="0.006656" />
+      </inertial>
+    </link>
+  </xacro:macro>
+  <gazebo>
+    <plugin name="p3d_base_controller" filename="libgazebo_ros_p3d.so">
+      <alwaysOn>true</alwaysOn>
+      <updateRate>50.0</updateRate>
+      <bodyName>base_link</bodyName>
+      <topicName>ground_truth/state</topicName>
+      <gaussianNoise>0.01</gaussianNoise>
+      <frameName>world</frameName>
+      <xyzOffsets>0 0 0</xyzOffsets>
+      <rpyOffsets>0 0 0</rpyOffsets>
+    </plugin>
+  </gazebo>
 </robot>
